Commit message: updated inertia values of ur5 model

File: universal-robot-ur5/ur5robot.urdf (robot description, URDF)
Before this commit: robot universal-robot-ur5, 9 links, 8 joints
Joints:
- joint elbow_joint: limit lower=-6.2831853 upper=6.2831853 effort=10.0 velocity=3.14159265 -> lower=-6.2831853 upper=6.2831853 effort=150.0 velocity=3.14159265
- joint shoulder_lift_joint: limit lower=-6.2831853 upper=6.2831853 effort=10.0 velocity=3.14159265 -> lower=-6.2831853 upper=6.2831853 effort=150.0 velocity=3.14159265
- joint shoulder_pan_joint: limit lower=-6.2831853 upper=6.2831853 effort=10.0 velocity=3.14159265 -> lower=-6.2831853 upper=6.2831853 effort=150.0 velocity=3.14159265
- joint wrist_1_joint: limit lower=-3.14159265 upper=0.7853981625 effort=10.0 velocity=3.14159265 -> lower=-3.14159265 upper=0.7853981625 effort=28.0 velocity=3.14159265
- joint wrist_2_joint: limit lower=-3.14159265 upper=3.14159265 effort=10.0 velocity=3.14159265 -> lower=-3.14159265 upper=3.14159265 effort=28.0 velocity=3.14159265
- joint wrist_3_joint: limit lower=-3.14159265 upper=3.14159265 effort=10.0 velocity=3.14159265 -> lower=-3.14159265 upper=3.14159265 effort=28.0 velocity=3.14159265

Commit message: set offset for base link

File: universal-robot-ur5/ur5robot.urdf (robot description, URDF)
Before this commit: robot universal-robot-ur5, 9 links, 8 joints
Joints:
- joint fixed: origin (none) -> xyz=0.0 0.0 0.1 rpy=0.0 0.0 0.0

Commit message: set baselink offset to be near the plane

File: universal-robot-ur5/ur5robot.urdf (robot description, URDF)
Before this commit: robot universal-robot-ur5, 9 links, 8 joints
Joints:
- joint fixed: origin xyz=0.0 0.0 0.1 rpy=0.0 0.0 0.0 -> xyz=0.0 0.0 0.01 rpy=0.0 0.0 0.0

Commit message: updated end effector inertial specifications

File: universal-robot-ur5/ur5robot.urdf (robot description, URDF)
Before this commit: robot universal-robot-ur5, 9 links, 8 joints
Links:
- link ee_link: mass None -> 0; geometry collision box size=0.05 0.05 0.05; visual box size=0.05 0.05 0.05

Commit message: corrected end effector joint and link

File: universal-robot-ur5/ur5robot.urdf (robot description, URDF)
Before this commit: robot universal-robot-ur5, 9 links, 8 joints
Links:
- link ee_link: mass 0 -> 5
Joints:
- removed joint fixed
- added joint world_base_joint: type fixed, parent world, child base_link, origin xyz=0.0 0.0 0.01 rpy=0.0 0.0 0.0
- joint ee_fixed_joint: axis (none) -> 0 1 0; limit (none) -> lower=0 upper=0 effort=0.0 velocity=0; type fixed -> revolute

Commit message: changed end-effector mass value so that the cube appears.

File: universal-robot-ur5/ur5robot.urdf (robot description, URDF)
Before this commit: robot universal-robot-ur5, 9 links, 8 joints
Links:
- link ee_link: mass 5 -> 0.00001

Commit message: changed joint limits

File: universal-robot-ur5/ur5robot.urdf (robot description, URDF)
Before this commit: robot universal-robot-ur5, 9 links, 8 joints
Joints:
- joint wrist_1_joint: limit lower=-3.14159265 upper=0.7853981625 effort=28.0 velocity=3.14159265 -> lower=-3.14159265 upper=4.71 effort=28.0 velocity=3.14159265
- joint wrist_2_joint: limit lower=-3.14159265 upper=3.14159265 effort=28.0 velocity=3.14159265 -> lower=-3.14159265 upper=4.71 effort=28.0 velocity=3.14159265
