Commit message: changed boris model slightly

File: boris-ft/model.urdf (robot description, URDF)
Before this commit: robot boris-ft, 23 links, 22 joints
Joints:
- joint left_lwr_arm_ft_sensor_joint: type revolute -> fixed

Commit message: added foot to boris model

File: boris-ft/model.urdf (robot description, URDF)
Before this commit: robot boris-ft, 23 links, 22 joints
Links:
- removed link left_lwr_tool
- removed link right_lwr_tool
- added link left_lwr_ft_link, mass 0.255; collision cylinder length=0.0333 radius=0.037; visual cylinder length=0.0333 radius=0.037
- added link left_lwr_tool_link, mass 0.255; collision mesh filename=model://boris-ft/meshes/boris-foot-white.stl scale=1 1 1; visual mesh filename=model://boris-ft/meshes/boris-foot-white.stl scale=1 1 1
- added link right_lwr_ft_link, mass 0.255; collision cylinder length=0.0333 radius=0.037; visual cylinder length=0.0333 radius=0.037
Joints:
- added joint left_lwr_ft_sensor_tool_joint: type fixed, parent left_lwr_ft_link, child left_lwr_tool_link, origin xyz=0 0 0.075 rpy=0 0 0, limit lower=0 upper=0 effort=0 velocity=0
- joint left_lwr_arm_ft_sensor_joint: child left_lwr_tool -> left_lwr_ft_link; type revolute -> fixed
- joint right_lwr_arm_ft_sensor_joint: child right_lwr_tool -> right_lwr_ft_link

Commit message: update boris and kuka models with foot

File: boris-ft/model.urdf (robot description, URDF)
Before this commit: robot boris-ft, 24 links, 23 joints
Links:
- link left_lwr_tool_link: mass 0.255 -> 0.1

File: kuka-lwr-4plus/model.urdf (robot description, URDF)
Before this commit: robot kuka-lwr, 9 links, 8 joints
Links:
- added link left_lwr_ft_link, mass 0.255; collision cylinder length=0.0333 radius=0.037; visual cylinder length=0.0333 radius=0.037
- added link left_lwr_tool_link, mass 0.1; collision mesh filename=model://boris-ft/meshes/boris-foot-white.stl scale=1 1 1; visual mesh filename=model://boris-ft/meshes/boris-foot-white.stl scale=1 1 1
Joints:
- added joint left_lwr_arm_ft_sensor_joint: type fixed, parent lwr_arm_7_link, child left_lwr_ft_link, origin xyz=0 0 0.0333 rpy=0 0 0, limit lower=0 upper=0 effort=0 velocity=0
- added joint left_lwr_ft_sensor_tool_joint: type fixed, parent left_lwr_ft_link, child left_lwr_tool_link, origin xyz=0 0 0.075 rpy=0 0 0, limit lower=0 upper=0 effort=0 velocity=0

Commit message: add sponge tool to right boris arm

File: boris-ft/model.urdf (robot description, URDF)
Before this commit: robot boris-ft, 24 links, 23 joints
Links:
- added link right_lwr_tool_link, mass 0.255; collision mesh filename=model://boris-ft/meshes/boris-foot-white.stl scale=1 1 1; visual mesh filename=model://boris-ft/meshes/boris-foot-white.stl scale=1 1 1
Joints:
- added joint right_lwr_ft_sensor_tool_joint: type fixed, parent right_lwr_ft_link, child right_lwr_tool_link, origin xyz=0 0 0.075 rpy=0 0 0, limit lower=0 upper=0 effort=0 velocity=0
- joint right_lwr_arm_ft_sensor_joint: type revolute -> fixed
