Commit message: adjusting the coman urdf to properly show in gazebo

File: iit-coman-no-forearms/model.urdf (robot description, URDF)
Before this commit: robot coman, 48 links, 47 joints
Links:
- link DWL: geometry collision mesh filename=model://iit-coman-no-forearms/meshes/simple/Torso1.STL scale=0.03937 0.03937 0.03937; visual mesh filename=model://iit-coman-no-forearms/meshes/Torso1.STL scale=0.03937 0.03937 0.03937
- link DWS: geometry collision mesh filename=model://iit-coman-no-forearms/meshes/simple/Torso2.STL scale=0.03937 0.03937 0.03937; visual mesh filename=model://iit-coman-no-forearms/meshes/Torso2.STL scale=0.03937 0.03937 0.03937
- link DWYTorso: geometry collision mesh filename=model://iit-coman-no-forearms/meshes/simple/Torso3.STL scale=0.03937 0.03937 0.03937; visual mesh filename=model://iit-coman-no-forearms/meshes/Torso3.STL scale=0.03937 0.03937 0.03937
- link LElb: geometry collision mesh filename=model://iit-coman-no-forearms/meshes/simple/Elbow.STL scale=1.0 1.0 1.0; visual mesh filename=model://iit-coman-no-forearms/meshes/Elbow.STL scale=1.0 1.0 1.0
- link LFoot: geometry collision mesh filename=model://iit-coman-no-forearms/meshes/simple/RoundFoot.STL scale=0.03937 -0.03937 0.03937; visual mesh filename=model://iit-coman-no-forearms/meshes/RoundFoot.STL scale=0.03937 -0.03937 0.03937
- link LFootmot: geometry collision mesh filename=model://iit-coman-no-forearms/meshes/simple/Leg4.STL scale=0.03937 -0.03937 0.03937; visual mesh filename=model://iit-coman-no-forearms/meshes/Leg4.STL scale=0.03937 -0.03937 0.03937
- link LForearm: geometry collision mesh filename=model://iit-coman-no-forearms/meshes/simple/ForearmOld.STL scale=0.03937 0.03937 0.03937; visual mesh filename=model://iit-coman-no-forearms/meshes/ForearmOld.STL scale=0.03937 0.03937 0.03937
- link LHipMot: geometry collision mesh filename=model://iit-coman-no-forearms/meshes/simple/Leg0.STL scale=0.03937 -0.03937 0.03937; visual mesh filename=model://iit-coman-no-forearms/meshes/Leg0.STL scale=0.03937 -0.03937 0.03937
- link LLowLeg: geometry collision mesh filename=model://iit-coman-no-forearms/meshes/simple/Leg3.STL scale=0.03937 -0.03937 0.03937; visual mesh filename=model://iit-coman-no-forearms/meshes/Leg3.STL scale=0.03937 -0.03937 0.03937
- link LShp: geometry collision mesh filename=model://iit-coman-no-forearms/meshes/simple/Arm0.STL scale=0.03937 -0.03937 0.03937; visual mesh filename=model://iit-coman-no-forearms/meshes/Arm0.STL scale=0.03937 -0.03937 0.03937
- link LShr: geometry collision mesh filename=model://iit-coman-no-forearms/meshes/simple/Arm1.STL scale=0.03937 -0.03937 0.03937; visual mesh filename=model://iit-coman-no-forearms/meshes/Arm1.STL scale=0.03937 -0.03937 0.03937
- link LShy: geometry collision mesh filename=model://iit-coman-no-forearms/meshes/simple/Arm2.STL scale=0.03937 -0.03937 0.03937; visual mesh filename=model://iit-coman-no-forearms/meshes/Arm2.STL scale=0.03937 -0.03937 0.03937
- link LThighLowLeg: geometry collision mesh filename=model://iit-coman-no-forearms/meshes/simple/Leg2.STL scale=0.03937 -0.03937 0.03937; visual mesh filename=model://iit-coman-no-forearms/meshes/Leg2.STL scale=0.03937 -0.03937 0.03937
- link LThighUpLeg: geometry collision mesh filename=model://iit-coman-no-forearms/meshes/simple/Leg1.STL scale=0.03937 -0.03937 0.03937; visual mesh filename=model://iit-coman-no-forearms/meshes/Leg1.STL scale=0.03937 -0.03937 0.03937
- link RElb: geometry collision mesh filename=model://iit-coman-no-forearms/meshes/simple/Elbow.STL scale=1.0 1.0 1.0; visual mesh filename=model://iit-coman-no-forearms/meshes/Elbow.STL scale=1.0 1.0 1.0
- link RFoot: geometry collision mesh filename=model://iit-coman-no-forearms/meshes/simple/RoundFoot.STL scale=0.03937 0.03937 0.03937; visual mesh filename=model://iit-coman-no-forearms/meshes/RoundFoot.STL scale=0.03937 0.03937 0.03937
- link RFootmot: geometry collision mesh filename=model://iit-coman-no-forearms/meshes/simple/Leg4.STL scale=0.03937 0.03937 0.03937; visual mesh filename=model://iit-coman-no-forearms/meshes/Leg4.STL scale=0.03937 0.03937 0.03937
- link RForearm: geometry collision mesh filename=model://iit-coman-no-forearms/meshes/simple/ForearmOld.STL scale=0.03937 0.03937 0.03937; visual mesh filename=model://iit-coman-no-forearms/meshes/ForearmOld.STL scale=0.03937 0.03937 0.03937
- link RHipMot: geometry collision mesh filename=model://iit-coman-no-forearms/meshes/simple/Leg0.STL scale=0.03937 0.03937 0.03937; visual mesh filename=model://iit-coman-no-forearms/meshes/Leg0.STL scale=0.03937 0.03937 0.03937
- link RLowLeg: geometry collision mesh filename=model://iit-coman-no-forearms/meshes/simple/Leg3.STL scale=0.03937 0.03937 0.03937; visual mesh filename=model://iit-coman-no-forearms/meshes/Leg3.STL scale=0.03937 0.03937 0.03937
- link RShp: geometry collision mesh filename=model://iit-coman-no-forearms/meshes/simple/Arm0.STL scale=0.03937 0.03937 0.03937; visual mesh filename=model://iit-coman-no-forearms/meshes/Arm0.STL scale=0.03937 0.03937 0.03937
- link RShr: geometry collision mesh filename=model://iit-coman-no-forearms/meshes/simple/Arm1.STL scale=0.03937 0.03937 0.03937; visual mesh filename=model://iit-coman-no-forearms/meshes/Arm1.STL scale=0.03937 0.03937 0.03937
- link RShy: geometry collision mesh filename=model://iit-coman-no-forearms/meshes/simple/Arm2.STL scale=0.03937 0.03937 0.03937; visual mesh filename=model://iit-coman-no-forearms/meshes/Arm2.STL scale=0.03937 0.03937 0.03937
- link RThighLowLeg: geometry collision mesh filename=model://iit-coman-no-forearms/meshes/simple/Leg2.STL scale=0.03937 0.03937 0.03937; visual mesh filename=model://iit-coman-no-forearms/meshes/Leg2.STL scale=0.03937 0.03937 0.03937
- link RThighUpLeg: geometry collision mesh filename=model://iit-coman-no-forearms/meshes/simple/Leg1.STL scale=0.03937 0.03937 0.03937; visual mesh filename=model://iit-coman-no-forearms/meshes/Leg1.STL scale=0.03937 0.03937 0.03937
- link Waist: geometry collision mesh filename=model://iit-coman-no-forearms/meshes/simple/Waist.STL scale=0.03937 0.03937 0.03937; visual mesh filename=model://iit-coman-no-forearms/meshes/Waist.STL scale=0.03937 0.03937 0.03937

Commit message: Added ft sensors

File: iit-coman-no-forearms/model.urdf (robot description, URDF)
Before this commit: robot coman, 48 links, 47 joints
Links:
- link DWL: geometry collision mesh filename=package://coman_urdf/meshes/simple/Torso1.STL scale=0.03937 0.03937 0.03937; visual mesh filename=package://coman_urdf/meshes/Torso1.STL scale=0.03937 0.03937 0.03937
- link DWS: geometry collision mesh filename=package://coman_urdf/meshes/simple/Torso2.STL scale=0.03937 0.03937 0.03937; visual mesh filename=package://coman_urdf/meshes/Torso2.STL scale=0.03937 0.03937 0.03937
- link DWYTorso: geometry collision mesh filename=package://coman_urdf/meshes/simple/Torso3.STL scale=0.03937 0.03937 0.03937; visual mesh filename=package://coman_urdf/meshes/Torso3.STL scale=0.03937 0.03937 0.03937
- link LElb: geometry collision mesh filename=package://coman_urdf/meshes/simple/Elbow.STL scale=1.0 1.0 1.0; visual mesh filename=package://coman_urdf/meshes/Elbow.STL scale=1.0 1.0 1.0
- link LFoot: geometry collision mesh filename=package://coman_urdf/meshes/simple/RoundFoot.STL scale=0.03937 -0.03937 0.03937; visual mesh filename=package://coman_urdf/meshes/RoundFoot.STL scale=0.03937 -0.03937 0.03937
- link LFootmot: geometry collision mesh filename=package://coman_urdf/meshes/simple/Leg4.STL scale=0.03937 -0.03937 0.03937; visual mesh filename=package://coman_urdf/meshes/Leg4.STL scale=0.03937 -0.03937 0.03937
- link LForearm: geometry collision mesh filename=package://coman_urdf/meshes/simple/ForearmOld.STL scale=0.03937 0.03937 0.03937; visual mesh filename=package://coman_urdf/meshes/ForearmOld.STL scale=0.03937 0.03937 0.03937
- link LHipMot: geometry collision mesh filename=package://coman_urdf/meshes/simple/Leg0.STL scale=0.03937 -0.03937 0.03937; visual mesh filename=package://coman_urdf/meshes/Leg0.STL scale=0.03937 -0.03937 0.03937
- link LLowLeg: geometry collision mesh filename=package://coman_urdf/meshes/simple/Leg3.STL scale=0.03937 -0.03937 0.03937; visual mesh filename=package://coman_urdf/meshes/Leg3.STL scale=0.03937 -0.03937 0.03937
- link LShp: geometry collision mesh filename=package://coman_urdf/meshes/simple/Arm0.STL scale=0.03937 -0.03937 0.03937; visual mesh filename=package://coman_urdf/meshes/Arm0.STL scale=0.03937 -0.03937 0.03937
- link LShr: geometry collision mesh filename=package://coman_urdf/meshes/simple/Arm1.STL scale=0.03937 -0.03937 0.03937; visual mesh filename=package://coman_urdf/meshes/Arm1.STL scale=0.03937 -0.03937 0.03937
- link LShy: geometry collision mesh filename=package://coman_urdf/meshes/simple/Arm2.STL scale=0.03937 -0.03937 0.03937; visual mesh filename=package://coman_urdf/meshes/Arm2.STL scale=0.03937 -0.03937 0.03937
- link LThighLowLeg: geometry collision mesh filename=package://coman_urdf/meshes/simple/Leg2.STL scale=0.03937 -0.03937 0.03937; visual mesh filename=package://coman_urdf/meshes/Leg2.STL scale=0.03937 -0.03937 0.03937
- link LThighUpLeg: geometry collision mesh filename=package://coman_urdf/meshes/simple/Leg1.STL scale=0.03937 -0.03937 0.03937; visual mesh filename=package://coman_urdf/meshes/Leg1.STL scale=0.03937 -0.03937 0.03937
- link RElb: geometry collision mesh filename=package://coman_urdf/meshes/simple/Elbow.STL scale=1.0 1.0 1.0; visual mesh filename=package://coman_urdf/meshes/Elbow.STL scale=1.0 1.0 1.0
- link RFoot: geometry collision mesh filename=package://coman_urdf/meshes/simple/RoundFoot.STL scale=0.03937 0.03937 0.03937; visual mesh filename=package://coman_urdf/meshes/RoundFoot.STL scale=0.03937 0.03937 0.03937
- link RFootmot: geometry collision mesh filename=package://coman_urdf/meshes/simple/Leg4.STL scale=0.03937 0.03937 0.03937; visual mesh filename=package://coman_urdf/meshes/Leg4.STL scale=0.03937 0.03937 0.03937
- link RForearm: geometry collision mesh filename=package://coman_urdf/meshes/simple/ForearmOld.STL scale=0.03937 0.03937 0.03937; visual mesh filename=package://coman_urdf/meshes/ForearmOld.STL scale=0.03937 0.03937 0.03937
- link RHipMot: geometry collision mesh filename=package://coman_urdf/meshes/simple/Leg0.STL scale=0.03937 0.03937 0.03937; visual mesh filename=package://coman_urdf/meshes/Leg0.STL scale=0.03937 0.03937 0.03937
- link RLowLeg: geometry collision mesh filename=package://coman_urdf/meshes/simple/Leg3.STL scale=0.03937 0.03937 0.03937; visual mesh filename=package://coman_urdf/meshes/Leg3.STL scale=0.03937 0.03937 0.03937
- link RShp: geometry collision mesh filename=package://coman_urdf/meshes/simple/Arm0.STL scale=0.03937 0.03937 0.03937; visual mesh filename=package://coman_urdf/meshes/Arm0.STL scale=0.03937 0.03937 0.03937
- link RShr: geometry collision mesh filename=package://coman_urdf/meshes/simple/Arm1.STL scale=0.03937 0.03937 0.03937; visual mesh filename=package://coman_urdf/meshes/Arm1.STL scale=0.03937 0.03937 0.03937
- link RShy: geometry collision mesh filename=package://coman_urdf/meshes/simple/Arm2.STL scale=0.03937 0.03937 0.03937; visual mesh filename=package://coman_urdf/meshes/Arm2.STL scale=0.03937 0.03937 0.03937
- link RThighLowLeg: geometry collision mesh filename=package://coman_urdf/meshes/simple/Leg2.STL scale=0.03937 0.03937 0.03937; visual mesh filename=package://coman_urdf/meshes/Leg2.STL scale=0.03937 0.03937 0.03937
- link RThighUpLeg: geometry collision mesh filename=package://coman_urdf/meshes/simple/Leg1.STL scale=0.03937 0.03937 0.03937; visual mesh filename=package://coman_urdf/meshes/Leg1.STL scale=0.03937 0.03937 0.03937
- link Waist: geometry collision mesh filename=package://coman_urdf/meshes/simple/Waist.STL scale=0.03937 0.03937 0.03937; visual mesh filename=package://coman_urdf/meshes/Waist.STL scale=0.03937 0.03937 0.03937
