Commit message: fixed errors in mesh paths caused by folder renaming

File: festo-axis/model.urdf (robot description, URDF)
Before this commit: robot festo-axis, 3 links, 2 joints
Links:
- link axis_link: geometry collision box size=0.196 1.422 0.1505; visual mesh filename=model://festo-axis/meshes/axis.dae
- link slide_link: geometry collision box size=0.179 0.290 0.0565; visual mesh filename=model://festo-axis/meshes/slide.dae scale=1 1 1

File: kuka-festo-8dof/model.urdf (robot description, URDF)
Before this commit: robot kuka-festo-8dof, 11 links, 10 joints
Links:
- link axis_link: geometry collision box size=0.196 1.422 0.1505; visual mesh filename=model://kuka-festo-8dof/meshes/axis.dae
- link lwr_arm_1_link: geometry collision mesh filename=model://kuka-festo-8dof/meshes/convex/arm_segment_a_convex.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 scale=1.0 1.0 1.0; visual mesh filename=model://kuka-festo-8dof/meshes/arm_segment_a.dae scale=100 100 100
- link lwr_arm_2_link: geometry collision mesh filename=model://kuka-festo-8dof/meshes/convex/arm_segment_b_convex.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 scale=1.0 1.0 1.0; visual mesh filename=model://kuka-festo-8dof/meshes/arm_segment_b.dae scale=100 100 100
- link lwr_arm_3_link: geometry collision mesh filename=model://kuka-festo-8dof/meshes/convex/arm_segment_a_convex.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 scale=1.0 1.0 1.0; visual mesh filename=model://kuka-festo-8dof/meshes/arm_segment_a.dae scale=100 100 100
- link lwr_arm_4_link: geometry collision mesh filename=model://kuka-festo-8dof/meshes/convex/arm_segment_b_convex.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 scale=1.0 1.0 1.0; visual mesh filename=model://kuka-festo-8dof/meshes/arm_segment_b.dae scale=100 100 100
- link lwr_arm_5_link: geometry collision mesh filename=model://kuka-festo-8dof/meshes/convex/arm_segment_last_conv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 scale=1.0 1.0 1.0; visual mesh filename=model://kuka-festo-8dof/meshes/arm_segment_last.dae scale=100 100 100
- link lwr_arm_6_link: geometry collision mesh filename=model://kuka-festo-8dof/meshes/convex/arm_wrist_convex.stl scale=1.0 1.0 1.0; visual mesh filename=model://kuka-festo-8dof/meshes/arm_wrist.dae scale=100 100 100
- link lwr_arm_7_link: geometry collision mesh filename=model://kuka-festo-8dof/meshes/arm_flanche.dae scale=100 100 100; visual mesh filename=model://kuka-festo-8dof/meshes/arm_flanche.dae scale=100 100 100
- link lwr_arm_base_link: geometry collision mesh filename=model://kuka-festo-8dof/meshes/convex/arm_base_convex.stl scale=0.9 0.9 0.9; visual mesh filename=model://kuka-festo-8dof/meshes/arm_base.dae scale=100 100 100
- link slide_link: geometry collision box size=0.179 0.290 0.0565; visual mesh filename=model://kuka-festo-8dof/meshes/slide.dae scale=1 1 1
Joints:
- joint axis_slide_joint: limit lower=-0.5 upper=0.5 effort=204 velocity=1.91986217719 -> lower=-0.35 upper=0.35 effort=204 velocity=1.91986217719
