Commit message: Updated models

File: iit-coman-hardware/model.urdf (robot description, URDF)
Before this commit: robot coman, 64 links, 63 joints
Links:
- added link LSoftHandFingers, mass 0.3; collision box size=0.07 0.01 0.07; visual box size=0.07 0.01 0.07
- added link RSoftHandFingers, mass 0.3; collision box size=0.07 0.01 0.07; visual box size=0.07 0.01 0.07
- link LSoftHand: geometry collision box size=0.07 0.01 0.07; visual box size=0.07 0.01 0.07
- link RSoftHand: geometry collision box size=0.07 0.01 0.07; visual box size=0.07 0.01 0.07
Joints:
- added joint l_handj2: type prismatic, parent LSoftHand, child LSoftHandFingers, origin xyz=0 -0.06 0.0 rpy=0 0 0, axis 0 1 0, limit lower=0.0 upper=0.05 effort=50 velocity=4.0
- added joint r_handj2: type prismatic, parent RSoftHand, child RSoftHandFingers, origin xyz=0 0.06 0.0 rpy=0 0 0, axis 0 1 0, limit lower=-0.05 upper=0.0 effort=50 velocity=4.0
- joint l_handj: axis -1 0 0 -> (none); limit lower=0.0 upper=1.57075 effort=5 velocity=4.0 -> (none); origin xyz=0 0 -0.04 rpy=0 0 0 -> xyz=0 0.03 -0.07 rpy=0 0 0; type revolute -> fixed
- joint r_handj: axis 1 0 0 -> (none); limit lower=0.0 upper=1.57075 effort=5 velocity=4.0 -> (none); origin xyz=0 0 -0.04 rpy=0 0 0 -> xyz=0 -0.03 -0.07 rpy=0 0 0; type revolute -> fixed

Commit message: Changed imu joint and added ft sensors

File: iit-coman-hardware/model.urdf (robot description, URDF)
Before this commit: robot coman, 66 links, 65 joints
Joints:
- joint imu_joint: origin xyz=-0.072 -0.0068 0.044 rpy=0 0 0 -> xyz=-0.072 -0.0068 0.044 rpy=1.57079632679 0 1.57079632679
- joint l_handj2: limit lower=0.0 upper=0.05 effort=50 velocity=4.0 -> lower=0.0 upper=10.0 effort=50 velocity=4.0
- joint r_handj2: limit lower=-0.05 upper=0.0 effort=50 velocity=4.0 -> lower=0.0 upper=10.0 effort=50 velocity=4.0

File: iit-coman-lowerbody-only/model.urdf (robot description, URDF)
Before this commit: robot coman, 31 links, 30 joints
Joints:
- joint imu_joint: origin xyz=-0.072 -0.0068 0.044 rpy=0 0 0 -> xyz=-0.072 -0.0068 0.044 rpy=1.57079632679 0 1.57079632679

File: iit-coman-no-forearms/model.urdf (robot description, URDF)
Before this commit: robot coman, 48 links, 47 joints
Joints:
- joint imu_joint: origin xyz=-0.072 -0.0068 0.044 rpy=0 0 0 -> xyz=-0.072 -0.0068 0.044 rpy=1.57079632679 0 1.57079632679

File: iit-coman/model.urdf (robot description, URDF)
Before this commit: robot coman, 64 links, 63 joints
Joints:
- joint imu_joint: origin xyz=-0.072 -0.0068 0.044 rpy=0 0 0 -> xyz=-0.072 -0.0068 0.044 rpy=1.57079632679 0 1.57079632679

Commit message: changed orientation jont left hand

File: iit-coman-hardware/model.urdf (robot description, URDF)
Before this commit: robot coman, 66 links, 65 joints
Joints:
- joint r_handj2: axis 0 1 0 -> 0 -1 0

Commit message: Updated model hardware with simple gripper and ros_imu plugin

File: iit-coman-hardware/model.urdf (robot description, URDF)
Before this commit: robot coman, 66 links, 65 joints
Joints:
- joint l_handj2: limit lower=0.0 upper=10.0 effort=50 velocity=4.0 -> lower=0.0 upper=0.05 effort=50 velocity=4.0
- joint r_handj2: limit lower=0.0 upper=10.0 effort=50 velocity=4.0 -> lower=0.0 upper=0.05 effort=50 velocity=4.0

Commit message: changed path to mesh

File: iit-coman-hardware/model.urdf (robot description, URDF)
Before this commit: robot coman, 66 links, 65 joints
Links:
- link DWL: geometry collision mesh filename=model://iit-coman-hardware/meshes/simple/Torso1.STL scale=0.03937 0.03937 0.03937; visual mesh filename=model://iit-coman-hardware/meshes/Torso1.STL scale=0.03937 0.03937 0.03937
- link DWS: geometry collision mesh filename=model://iit-coman-hardware/meshes/simple/Torso2.STL scale=0.03937 0.03937 0.03937; visual mesh filename=model://iit-coman-hardware/meshes/Torso2.STL scale=0.03937 0.03937 0.03937
- link DWYTorso: geometry collision mesh filename=model://iit-coman-hardware/meshes/simple/Torso3.STL scale=0.03937 0.03937 0.03937; visual mesh filename=model://iit-coman-hardware/meshes/Torso3.STL scale=0.03937 0.03937 0.03937
- link LElb: geometry collision mesh filename=model://iit-coman-hardware/meshes/simple/Elbow.STL scale=1.0 1.0 1.0; visual mesh filename=model://iit-coman-hardware/meshes/Elbow.STL scale=1.0 1.0 1.0
- link LFootmot: geometry collision mesh filename=model://iit-coman-hardware/meshes/simple/Leg4.STL scale=0.03937 -0.03937 0.03937; visual mesh filename=model://iit-coman-hardware/meshes/Leg4.STL scale=0.03937 -0.03937 0.03937
- link LForearm: geometry collision mesh filename=model://iit-coman-hardware/meshes/simple/Forearm0.STL scale=1.0 1.0 1.0; visual mesh filename=model://iit-coman-hardware/meshes/Forearm0.STL scale=0.1 0.1 0.1
- link LHipMot: geometry collision mesh filename=model://iit-coman-hardware/meshes/simple/Leg0.STL scale=0.03937 -0.03937 0.03937; visual mesh filename=model://iit-coman-hardware/meshes/Leg0.STL scale=0.03937 -0.03937 0.03937
- link LLowLeg: geometry collision mesh filename=model://iit-coman-hardware/meshes/simple/Leg3.STL scale=0.03937 -0.03937 0.03937; visual mesh filename=model://iit-coman-hardware/meshes/Leg3.STL scale=0.03937 -0.03937 0.03937
- link LShp: geometry collision mesh filename=model://iit-coman-hardware/meshes/simple/Arm0.STL scale=0.03937 -0.03937 0.03937; visual mesh filename=model://iit-coman-hardware/meshes/Arm0.STL scale=0.03937 -0.03937 0.03937
- link LShr: geometry collision mesh filename=model://iit-coman-hardware/meshes/simple/Arm1.STL scale=0.03937 -0.03937 0.03937; visual mesh filename=model://iit-coman-hardware/meshes/Arm1.STL scale=0.03937 -0.03937 0.03937
- link LShy: geometry collision mesh filename=model://iit-coman-hardware/meshes/simple/Arm2.STL scale=0.03937 -0.03937 0.03937; visual mesh filename=model://iit-coman-hardware/meshes/Arm2.STL scale=0.03937 -0.03937 0.03937
- link LThighLowLeg: geometry collision mesh filename=model://iit-coman-hardware/meshes/simple/Leg2.STL scale=0.03937 -0.03937 0.03937; visual mesh filename=model://iit-coman-hardware/meshes/Leg2.STL scale=0.03937 -0.03937 0.03937
- link LThighUpLeg: geometry collision mesh filename=model://iit-coman-hardware/meshes/simple/Leg1.STL scale=0.03937 -0.03937 0.03937; visual mesh filename=model://iit-coman-hardware/meshes/Leg1.STL scale=0.03937 -0.03937 0.03937
- link LWrMot2: geometry collision mesh filename=model://iit-coman-hardware/meshes/simple/Forearm1.STL scale=0.001 0.001 0.001; visual mesh filename=model://iit-coman-hardware/meshes/Forearm1.STL scale=0.001 0.001 0.001
- link LWrMot3: geometry collision mesh filename=model://iit-coman-hardware/meshes/simple/Forearm2.STL scale=0.001 0.001 0.001; visual mesh filename=model://iit-coman-hardware/meshes/Forearm2.STL scale=0.001 0.001 0.001
- link RElb: geometry collision mesh filename=model://iit-coman-hardware/meshes/simple/Elbow.STL scale=1.0 1.0 1.0; visual mesh filename=model://iit-coman-hardware/meshes/Elbow.STL scale=1.0 1.0 1.0
- link RFootmot: geometry collision mesh filename=model://iit-coman-hardware/meshes/simple/Leg4.STL scale=0.03937 0.03937 0.03937; visual mesh filename=model://iit-coman-hardware/meshes/Leg4.STL scale=0.03937 0.03937 0.03937
- link RForearm: geometry collision mesh filename=model://iit-coman-hardware/meshes/simple/Forearm0.STL scale=1.0 1.0 1.0; visual mesh filename=model://iit-coman-hardware/meshes/Forearm0.STL scale=0.1 0.1 0.1
- link RHipMot: geometry collision mesh filename=model://iit-coman-hardware/meshes/simple/Leg0.STL scale=0.03937 0.03937 0.03937; visual mesh filename=model://iit-coman-hardware/meshes/Leg0.STL scale=0.03937 0.03937 0.03937
- link RLowLeg: geometry collision mesh filename=model://iit-coman-hardware/meshes/simple/Leg3.STL scale=0.03937 0.03937 0.03937; visual mesh filename=model://iit-coman-hardware/meshes/Leg3.STL scale=0.03937 0.03937 0.03937
- link RShp: geometry collision mesh filename=model://iit-coman-hardware/meshes/simple/Arm0.STL scale=0.03937 0.03937 0.03937; visual mesh filename=model://iit-coman-hardware/meshes/Arm0.STL scale=0.03937 0.03937 0.03937
- link RShr: geometry collision mesh filename=model://iit-coman-hardware/meshes/simple/Arm1.STL scale=0.03937 0.03937 0.03937; visual mesh filename=model://iit-coman-hardware/meshes/Arm1.STL scale=0.03937 0.03937 0.03937
- link RShy: geometry collision mesh filename=model://iit-coman-hardware/meshes/simple/Arm2.STL scale=0.03937 0.03937 0.03937; visual mesh filename=model://iit-coman-hardware/meshes/Arm2.STL scale=0.03937 0.03937 0.03937
- link RThighLowLeg: geometry collision mesh filename=model://iit-coman-hardware/meshes/simple/Leg2.STL scale=0.03937 0.03937 0.03937; visual mesh filename=model://iit-coman-hardware/meshes/Leg2.STL scale=0.03937 0.03937 0.03937
- link RThighUpLeg: geometry collision mesh filename=model://iit-coman-hardware/meshes/simple/Leg1.STL scale=0.03937 0.03937 0.03937; visual mesh filename=model://iit-coman-hardware/meshes/Leg1.STL scale=0.03937 0.03937 0.03937
- link RWrMot2: geometry collision mesh filename=model://iit-coman-hardware/meshes/simple/Forearm1.STL scale=0.001 0.001 0.001; visual mesh filename=model://iit-coman-hardware/meshes/Forearm1.STL scale=0.001 0.001 0.001
- link RWrMot3: geometry collision mesh filename=model://iit-coman-hardware/meshes/simple/Forearm2.STL scale=0.001 0.001 0.001; visual mesh filename=model://iit-coman-hardware/meshes/Forearm2.STL scale=0.001 0.001 0.001
- link Waist: geometry collision mesh filename=model://iit-coman-hardware/meshes/simple/Waist.STL scale=0.03937 0.03937 0.03937; visual mesh filename=model://iit-coman-hardware/meshes/Waist.STL scale=0.03937 0.03937 0.03937
