Commit message: fixed broken 4plus model and names

File: kuka-lwr-4plus/model.urdf (robot description, URDF)
Before this commit: robot kuka-lwr, 11 links, 10 joints
Links:
- removed link left_lwr_ft_link
- removed link left_lwr_tool_link
Joints:
- removed joint left_lwr_arm_ft_sensor_joint
- removed joint left_lwr_ft_sensor_tool_joint

File: kuka-lwr-4plus/model_capsule_collision.urdf (robot description, URDF)
Before this commit: robot kuka-lwr-4plus-tool, 10 links, 9 joints
Links:
- removed link lwr_tool
- link lwr_arm_1_link: geometry collision cylinder length=0.30 radius=0.08; visual mesh filename=model://kuka-lwr-4plus/meshes/arm_segment_a.dae scale=100 100 100
- link lwr_arm_2_link: geometry collision cylinder length=0.30 radius=0.08; visual mesh filename=model://kuka-lwr-4plus/meshes/arm_segment_b.dae scale=100 100 100
- link lwr_arm_3_link: geometry collision cylinder length=0.30 radius=0.08; visual mesh filename=model://kuka-lwr-4plus/meshes/arm_segment_a.dae scale=100 100 100
- link lwr_arm_4_link: geometry collision cylinder length=0.30 radius=0.08; visual mesh filename=model://kuka-lwr-4plus/meshes/arm_segment_b.dae scale=100 100 100
- link lwr_arm_5_link: geometry collision cylinder length=0.263 radius=0.07; visual mesh filename=model://kuka-lwr-4plus/meshes/arm_segment_last.dae scale=100 100 100
- link lwr_arm_6_link: geometry collision cylinder length=0.132 radius=0.075; visual mesh filename=model://kuka-lwr-4plus/meshes/arm_wrist.dae scale=100 100 100
- link lwr_arm_7_link: geometry collision cylinder length=0.035 radius=0.05; visual mesh filename=model://kuka-lwr-4plus/meshes/arm_flanche.dae scale=100 100 100
- link lwr_arm_base_link: geometry collision cylinder length=0.11 radius=0.09; visual mesh filename=model://kuka-lwr-4plus/meshes/arm_base.dae scale=100 100 100
Joints:
- removed joint lwr_ft_sensor_joint
