Commit message: updated kuka with sponge with new foot design

File: kuka-lwr-4plus-sponge/model.urdf (robot description, URDF)
Before this commit: robot kuka-lwr, 11 links, 10 joints
Links:
- link lwr_tool_link: mass 0.255 -> 0.691; geometry collision mesh filename=model://kuka-lwr-4plus-sponge/NewKukaFoot.stl scale=1.0 1.0 1; visual mesh filename=model://kuka-lwr-4plus-sponge/NewKukaFoot.stl scale=1 1 1

Commit message: updated triangle and sponge model

File: kuka-lwr-4plus-sponge/model.urdf (robot description, URDF)
Before this commit: robot kuka-lwr-4plus-sponge, 11 links, 10 joints
Links:
- removed link lwr_ft_link
Joints:
- removed joint lwr_arm_ft_sensor_joint
- removed joint lwr_ft_sensor_tool_joint
- added joint lwr_arm_7_tool_joint: type fixed, parent lwr_arm_7_link, child lwr_tool_link, origin xyz=0 0 0.075 rpy=0 0 0, limit lower=0 upper=0 effort=0 velocity=0
