Commit message: Add inertial tags (WARNING: Values a totally irrealistic!)
This adds inertial tags for all link of the panda arm. Inertial values
are simply copied from the kuka-lwr-4plus model and thus probably not
very useful. However, Gazebo needs inertial tags in order to process
URDF files.

File: franka-panda-arm/model.urdf (robot description, URDF)
Before this commit: robot panda, 9 links, 8 joints
Links:
- link panda_link0: mass None -> 1.2
- link panda_link1: mass None -> 2.0
- link panda_link2: mass None -> 2.0
- link panda_link3: mass None -> 2.0
- link panda_link4: mass None -> 2.0
- link panda_link5: mass None -> 2.0
- link panda_link6: mass None -> 1.0
- link panda_link7: mass None -> 0.2

Commit message: Introduce rigid joint to world link
Basically mount the arm to the ground

File: franka-panda-arm/model.urdf (robot description, URDF)
Before this commit: robot panda, 9 links, 8 joints
Links:
- added link world
Joints:
- added joint panda_world_joint: type fixed, parent world, child panda_link0, origin xyz=0 0 0.01 rpy=0 0 0
