Commit message: Updated model with almost real hardware limits

File: iit-cogimon/model.urdf (robot description, URDF)
Before this commit: robot cogimon, 14 links, 13 joints
Links:
- added link l_ankle
- added link l_foot_lower_left_link
- added link l_foot_lower_right_link
- added link l_foot_upper_left_link
- added link l_foot_upper_right_link
- added link l_heel
- added link l_sole
- added link l_toe
- added link r_ankle
- added link r_foot_lower_left_link
- added link r_foot_lower_right_link
- added link r_foot_upper_left_link
- added link r_foot_upper_right_link
- added link r_heel
- added link r_sole
- added link r_toe
Joints:
- added joint l_ankle_joint: type fixed, parent LFoot, child l_ankle, origin xyz=0 0 0 rpy=0 0 0
- added joint l_foot_lower_left_joint: type fixed, parent l_sole, child l_foot_lower_left_link, origin xyz=-0.1035 0.055 0 rpy=0 0 0
- added joint l_foot_lower_right_joint: type fixed, parent l_sole, child l_foot_lower_right_link, origin xyz=-0.1035 -0.055 0 rpy=0 0 0
- added joint l_foot_upper_left_joint: type fixed, parent l_sole, child l_foot_upper_left_link, origin xyz=0.107 0.055 0 rpy=0 0 0
- added joint l_foot_upper_right_joint: type fixed, parent l_sole, child l_foot_upper_right_link, origin xyz=0.107 -0.055 0 rpy=0 0 0
- added joint l_heel_joint: type fixed, parent l_sole, child l_heel, origin xyz=-0.1035 0 0 rpy=0 0 0
- added joint l_sole_joint: type fixed, parent l_ankle, child l_sole, origin xyz=0 0 -0.054 rpy=0 0 0
- added joint l_toe_joint: type fixed, parent l_sole, child l_toe, origin xyz=0.107 0 0 rpy=0 0 0
- added joint r_ankle_joint: type fixed, parent RFoot, child r_ankle, origin xyz=0 0 0 rpy=0 0 0
- added joint r_foot_lower_left_joint: type fixed, parent r_sole, child r_foot_lower_left_link, origin xyz=-0.1035 0.055 0 rpy=0 0 0
- added joint r_foot_lower_right_joint: type fixed, parent r_sole, child r_foot_lower_right_link, origin xyz=-0.1035 -0.055 0 rpy=0 0 0
- added joint r_foot_upper_left_joint: type fixed, parent r_sole, child r_foot_upper_left_link, origin xyz=0.107 0.055 0 rpy=0 0 0
- added joint r_foot_upper_right_joint: type fixed, parent r_sole, child r_foot_upper_right_link, origin xyz=0.107 -0.055 0 rpy=0 0 0
- added joint r_heel_joint: type fixed, parent r_sole, child r_heel, origin xyz=-0.1035 0 0 rpy=0 0 0
- added joint r_sole_joint: type fixed, parent r_ankle, child r_sole, origin xyz=0 0 -0.054 rpy=0 0 0
- added joint r_toe_joint: type fixed, parent r_sole, child r_toe, origin xyz=0.107 0 0 rpy=0 0 0
- joint LAnklePitch: limit lower=-1.57079632679 upper=1.57079632679 effort=176 velocity=3.67 -> lower=-0.872664625995 upper=0.698131700796 effort=179 velocity=4.9
- joint LAnkleRoll: limit lower=-1.57079632679 upper=1.57079632679 effort=176 velocity=3.67 -> lower=-0.261799387798 upper=0.261799387798 effort=230 velocity=3.2
- joint LHipLat: limit lower=-1.57079632679 upper=1.57079632679 effort=176 velocity=3.67 -> lower=-0.523598775597 upper=1.65806278939 effort=235 velocity=7.4
- joint LHipSag: limit lower=-1.57079632679 upper=1.57079632679 effort=176 velocity=3.67 -> lower=-1.91986217719 upper=1.55334303427 effort=235 velocity=7.4
- joint LHipYaw: limit lower=-1.57079632679 upper=1.57079632679 effort=176 velocity=3.67 -> lower=-0.558505360637 upper=1.57079632679 effort=153 velocity=4.6
- joint LKneePitch: limit lower=-1.57079632679 upper=1.57079632679 effort=176 velocity=3.67 -> lower=0.0 upper=2.44346095279 effort=313 velocity=5.5
- joint RAnklePitch: limit lower=-1.57079632679 upper=1.57079632679 effort=176 velocity=3.67 -> lower=-0.872664625995 upper=0.698131700796 effort=179 velocity=4.9
- joint RAnkleRoll: limit lower=-1.57079632679 upper=1.57079632679 effort=176 velocity=3.67 -> lower=-0.261799387798 upper=0.261799387798 effort=230 velocity=3.2
- joint RHipLat: limit lower=-1.57079632679 upper=1.57079632679 effort=176 velocity=3.67 -> lower=-1.65806278939 upper=0.523598775597 effort=235 velocity=7.4
- joint RHipSag: limit lower=-1.57079632679 upper=1.57079632679 effort=176 velocity=3.67 -> lower=-1.91986217719 upper=1.55334303427 effort=235 velocity=7.4
- joint RHipYaw: limit lower=-1.57079632679 upper=1.57079632679 effort=176 velocity=3.67 -> lower=-1.57079632679 upper=0.558505360637 effort=153 velocity=4.9
- joint RKneePitch: limit lower=-1.57079632679 upper=1.57079632679 effort=176 velocity=3.67 -> lower=0.0 upper=2.44346095279 effort=313 velocity=5.5

Commit message: fix the path and type for meshes

File: iit-cogimon/model.urdf (robot description, URDF)
Before this commit: robot cogimon, 30 links, 29 joints
Links:
- link LFoot: geometry collision box size=0.21 0.11 0.015; visual mesh filename=model://iit-cogimon/meshes/Foot.stl scale=0.001 0.001 0.001
- link LFootmot: geometry collision mesh filename=model://iit-cogimon/meshes/simple/AnklePitch.stl scale=0.001 0.001 0.001; visual mesh filename=model://iit-cogimon/meshes/AnklePitch.stl scale=0.001 0.001 0.001
- link LHipMot: geometry collision mesh filename=model://iit-cogimon/meshes/simple/HipRoll.stl scale=0.001 0.001 0.001; visual mesh filename=model://iit-cogimon/meshes/HipRoll.stl scale=0.001 0.001 0.001
- link LLowLeg: geometry collision mesh filename=model://iit-cogimon/meshes/simple/KneePitch.stl scale=0.001 0.001 0.001; visual mesh filename=model://iit-cogimon/meshes/KneePitch.stl scale=0.001 0.001 0.001
- link LThighLowLeg: geometry collision mesh filename=model://iit-cogimon/meshes/simple/HipYaw.stl scale=0.001 0.001 0.001; visual mesh filename=model://iit-cogimon/meshes/HipYaw.stl scale=0.001 0.001 0.001
- link LThighUpLeg: geometry collision mesh filename=model://iit-cogimon/meshes/simple/HipPitch.stl scale=0.001 0.001 0.001; visual mesh filename=model://iit-cogimon/meshes/HipPitch.stl scale=0.001 0.001 0.001
- link RFoot: geometry collision box size=0.21 0.11 0.015; visual mesh filename=model://iit-cogimon/meshes/Foot.stl scale=0.001 0.001 0.001
- link RFootmot: geometry collision mesh filename=model://iit-cogimon/meshes/simple/AnklePitch.stl scale=0.001 0.001 0.001; visual mesh filename=model://iit-cogimon/meshes/AnklePitch.stl scale=0.001 0.001 0.001
- link RHipMot: geometry collision mesh filename=model://iit-cogimon/meshes/simple/HipRoll.stl scale=0.001 -0.001 0.001; visual mesh filename=model://iit-cogimon/meshes/HipRoll.stl scale=0.001 -0.001 0.001
- link RLowLeg: geometry collision mesh filename=model://iit-cogimon/meshes/simple/KneePitch.stl scale=0.001 -0.001 0.001; visual mesh filename=model://iit-cogimon/meshes/KneePitch.stl scale=0.001 -0.001 0.001
- link RThighLowLeg: geometry collision mesh filename=model://iit-cogimon/meshes/simple/HipYaw.stl scale=0.001 -0.001 0.001; visual mesh filename=model://iit-cogimon/meshes/HipYaw.stl scale=0.001 -0.001 0.001
- link RThighUpLeg: geometry collision mesh filename=model://iit-cogimon/meshes/simple/HipPitch.stl scale=0.001 -0.001 0.001; visual mesh filename=model://iit-cogimon/meshes/HipPitch.stl scale=0.001 -0.001 0.001
- link Waist: geometry collision mesh filename=model://iit-cogimon/meshes/simple/Waist.stl scale=0.001 0.001 0.001; visual mesh filename=model://iit-cogimon/meshes/Waist.stl scale=0.001 0.001 0.001

Commit message: Added ft sensors. updated gains

File: iit-cogimon/model.urdf (robot description, URDF)
Before this commit: robot cogimon, 30 links, 29 joints
Links:
- added link l_leg_ft
- added link r_leg_ft
- added link world
Joints:
- added joint l_leg_ft_joint: type fixed, parent LFoot, child l_leg_ft, origin xyz=0 0 -0.035 rpy=0 0 0
- added joint r_leg_ft_joint: type fixed, parent RFoot, child r_leg_ft, origin xyz=0 0 -0.035 rpy=0 0 0
- added joint reference: type floating, parent world, child base_link

Commit message: Added torso roll joint and bar

File: iit-cogimon/model.urdf (robot description, URDF)
Before this commit: robot cogimon, 33 links, 32 joints
Links:
- added link DWL, mass 7.4182685e-01; collision mesh filename=package://cogimon_urdf/meshes/simple/TorsoRoll.stl scale=0.001 0.001 0.001; visual mesh filename=package://cogimon_urdf/meshes/TorsoRoll.stl scale=0.001 0.001 0.001
- added link pennacchio, mass 2.1651618; collision mesh filename=package://cogimon_urdf/meshes/simple/Pennacchio.stl scale=0.001 0.001 0.001; visual mesh filename=package://cogimon_urdf/meshes/Pennacchio.stl scale=0.001 0.001 0.001
- link LFoot: geometry collision box size=0.21 0.11 0.015; visual mesh filename=package://cogimon_urdf/meshes/Foot.stl scale=0.001 0.001 0.001
- link LFootmot: geometry collision mesh filename=package://cogimon_urdf/meshes/simple/AnklePitch.stl scale=0.001 0.001 0.001; visual mesh filename=package://cogimon_urdf/meshes/AnklePitch.stl scale=0.001 0.001 0.001
- link LHipMot: geometry collision mesh filename=package://cogimon_urdf/meshes/simple/HipRoll.stl scale=0.001 0.001 0.001; visual mesh filename=package://cogimon_urdf/meshes/HipRoll.stl scale=0.001 0.001 0.001
- link LLowLeg: geometry collision mesh filename=package://cogimon_urdf/meshes/simple/KneePitch.stl scale=0.001 0.001 0.001; visual mesh filename=package://cogimon_urdf/meshes/KneePitch.stl scale=0.001 0.001 0.001
- link LThighLowLeg: geometry collision mesh filename=package://cogimon_urdf/meshes/simple/HipYaw.stl scale=0.001 0.001 0.001; visual mesh filename=package://cogimon_urdf/meshes/HipYaw.stl scale=0.001 0.001 0.001
- link LThighUpLeg: geometry collision mesh filename=package://cogimon_urdf/meshes/simple/HipPitch.stl scale=0.001 0.001 0.001; visual mesh filename=package://cogimon_urdf/meshes/HipPitch.stl scale=0.001 0.001 0.001
- link RFoot: geometry collision box size=0.21 0.11 0.015; visual mesh filename=package://cogimon_urdf/meshes/Foot.stl scale=0.001 0.001 0.001
- link RFootmot: geometry collision mesh filename=package://cogimon_urdf/meshes/simple/AnklePitch.stl scale=0.001 0.001 0.001; visual mesh filename=package://cogimon_urdf/meshes/AnklePitch.stl scale=0.001 0.001 0.001
- link RHipMot: geometry collision mesh filename=package://cogimon_urdf/meshes/simple/HipRoll.stl scale=0.001 -0.001 0.001; visual mesh filename=package://cogimon_urdf/meshes/HipRoll.stl scale=0.001 -0.001 0.001
- link RLowLeg: geometry collision mesh filename=package://cogimon_urdf/meshes/simple/KneePitch.stl scale=0.001 -0.001 0.001; visual mesh filename=package://cogimon_urdf/meshes/KneePitch.stl scale=0.001 -0.001 0.001
- link RThighLowLeg: geometry collision mesh filename=package://cogimon_urdf/meshes/simple/HipYaw.stl scale=0.001 -0.001 0.001; visual mesh filename=package://cogimon_urdf/meshes/HipYaw.stl scale=0.001 -0.001 0.001
- link RThighUpLeg: geometry collision mesh filename=package://cogimon_urdf/meshes/simple/HipPitch.stl scale=0.001 -0.001 0.001; visual mesh filename=package://cogimon_urdf/meshes/HipPitch.stl scale=0.001 -0.001 0.001
- link Waist: geometry collision mesh filename=package://cogimon_urdf/meshes/simple/Waist.stl scale=0.001 0.001 0.001; visual mesh filename=package://cogimon_urdf/meshes/Waist.stl scale=0.001 0.001 0.001
Joints:
- added joint WaistLat: type revolute, parent Waist, child DWL, origin xyz=0.012 0.0 0.0 rpy=0 0 0, axis 1 0 0, limit lower=-0.523598775597 upper=0.523598775597 effort=150 velocity=7.4
- added joint pennacchio_frame: type fixed, parent DWL, child pennacchio, origin xyz=-0.0540957 0.0 0.0665 rpy=0 0 0

Commit message: Updated model with extra weight

File: iit-cogimon/model.urdf (robot description, URDF)
Before this commit: robot cogimon, 35 links, 34 joints
Links:
- added link weight, mass 30.0; collision cylinder length=0.06 radius=0.055; visual cylinder length=0.06 radius=0.055
Joints:
- added joint weight_frame: type fixed, parent pennacchio, child weight, origin xyz=0. 0. 0.2 rpy=0 0 0

Commit message: Removed capsule files. Added missing stl. Updated urdf and srdf

File: iit-cogimon/model.urdf (robot description, URDF)
Before this commit: robot cogimon, 36 links, 35 joints
Links:
- removed link pennacchio
- removed link weight
- added link DWLExt, mass 9.6910635e-01; collision mesh filename=package://cogimon_urdf/meshes/simple/TorsoRollExt.stl scale=0.001 0.001 0.001; visual mesh filename=package://cogimon_urdf/meshes/TorsoRollExt.stl scale=0.001 0.001 0.001
- added link DWYTorso, mass 1.2512295e+01; collision mesh filename=package://cogimon_urdf/meshes/simple/Chest.stl scale=0.001 0.001 0.001; visual mesh filename=package://cogimon_urdf/meshes/Chest.stl scale=0.001 0.001 0.001
- added link LElb, mass 1.3157289; collision mesh filename=package://cogimon_urdf/meshes/simple/Elbow.STL scale=0.001 -0.001 0.001; visual mesh filename=package://cogimon_urdf/meshes/Elbow.STL scale=0.001 -0.001 0.001
- added link LForearm, mass 1.4908547; collision mesh filename=package://cogimon_urdf/meshes/simple/Forearm.STL scale=0.001 -0.001 0.001; visual mesh filename=package://cogimon_urdf/meshes/Forearm.STL scale=0.001 -0.001 0.001
- added link LShp, mass 1.9628675; collision mesh filename=package://cogimon_urdf/meshes/simple/ShoulderPitch.STL scale=0.001 -0.001 0.001; visual mesh filename=package://cogimon_urdf/meshes/ShoulderPitch.STL scale=0.001 -0.001 0.001
- added link LShr, mass 1.8595811; collision mesh filename=package://cogimon_urdf/meshes/simple/ShoulderRoll.STL scale=0.001 -0.001 0.001; visual mesh filename=package://cogimon_urdf/meshes/ShoulderRoll.STL scale=0.001 -0.001 0.001
- added link LShy, mass 1.6678109; collision mesh filename=package://cogimon_urdf/meshes/simple/ShoulderYaw.STL scale=0.001 -0.001 0.001; visual mesh filename=package://cogimon_urdf/meshes/ShoulderYaw.STL scale=0.001 -0.001 0.001
- added link LWrMot2, mass 1.1263612; collision mesh filename=package://cogimon_urdf/meshes/simple/ForearmPitch.STL scale=0.001 -0.001 0.001; visual mesh filename=package://cogimon_urdf/meshes/ForearmPitch.STL scale=0.001 -0.001 0.001
- added link LWrMot3, mass 2.7966428e-01; collision mesh filename=package://cogimon_urdf/meshes/simple/ForearmYaw.STL scale=0.001 -0.001 0.001; visual mesh filename=package://cogimon_urdf/meshes/ForearmYaw.STL scale=0.001 -0.001 0.001
- added link RElb, mass 1.3157289; collision mesh filename=package://cogimon_urdf/meshes/simple/Elbow.STL scale=0.001 0.001 0.001; visual mesh filename=package://cogimon_urdf/meshes/Elbow.STL scale=0.001 0.001 0.001
- added link RForearm, mass 1.4908547; collision mesh filename=package://cogimon_urdf/meshes/simple/Forearm.STL scale=0.001 0.001 0.001; visual mesh filename=package://cogimon_urdf/meshes/Forearm.STL scale=0.001 0.001 0.001
- added link RShp, mass 1.9628675; collision mesh filename=package://cogimon_urdf/meshes/simple/ShoulderPitch.STL scale=0.001 0.001 0.001; visual mesh filename=package://cogimon_urdf/meshes/ShoulderPitch.STL scale=0.001 0.001 0.001
- added link RShr, mass 1.8595811; collision mesh filename=package://cogimon_urdf/meshes/simple/ShoulderRoll.STL scale=0.001 0.001 0.001; visual mesh filename=package://cogimon_urdf/meshes/ShoulderRoll.STL scale=0.001 0.001 0.001
- added link RShy, mass 1.6678109; collision mesh filename=package://cogimon_urdf/meshes/simple/ShoulderYaw.STL scale=0.001 0.001 0.001; visual mesh filename=package://cogimon_urdf/meshes/ShoulderYaw.STL scale=0.001 0.001 0.001
- added link RWrMot2, mass 1.1263612; collision mesh filename=package://cogimon_urdf/meshes/simple/ForearmPitch.STL scale=0.001 0.001 0.001; visual mesh filename=package://cogimon_urdf/meshes/ForearmPitch.STL scale=0.001 0.001 0.001
- added link RWrMot3, mass 2.7966428e-01; collision mesh filename=package://cogimon_urdf/meshes/simple/ForearmYaw.STL scale=0.001 0.001 0.001; visual mesh filename=package://cogimon_urdf/meshes/ForearmYaw.STL scale=0.001 0.001 0.001
- added link imu_link, mass 0
Joints:
- removed joint pennacchio_frame
- removed joint weight_frame
- added joint LElbj: type revolute, parent LShy, child LElb, origin xyz=0.045 0.05515 -0.074 rpy=0 0 0, axis 0 1 0, limit lower=-2.492 upper=0.298 effort=147 velocity=6.283
- added joint LForearmPlate: type revolute, parent LElb, child LForearm, origin xyz=-0.015 -0.05515 -0.095 rpy=0 0 0, axis 0 0 1, limit lower=-2.55 upper=2.55 effort=55 velocity=6.283
- added joint LShLat: type revolute, parent LShp, child LShr, origin xyz=-0.09015 0.062 0 rpy=-0.1745327 0 0, axis 1 0 0, limit lower=0.037 upper=3.517 effort=120 velocity=6.283
- added joint LShSag: type revolute, parent DWYTorso, child LShp, origin xyz=0.0457475 0.169137 0.155126 rpy=0.174533 0 -0.5235988, axis 0 1 0, limit lower=-3.352 upper=1.603 effort=147 velocity=6.283
- added joint LShYaw: type revolute, parent LShr, child LShy, origin xyz=0.09015 0 -0.21815 rpy=0 0 0, axis 0 0 1, limit lower=-2.55 upper=2.55 effort=147 velocity=6.283
- added joint LWrj1: type revolute, parent LForearm, child LWrMot2, origin xyz=0 0.049 -0.156 rpy=0 0 0, axis 0 1 0, limit lower=-1.562 upper=1.478 effort=55 velocity=6.283
- added joint LWrj2: type revolute, parent LWrMot2, child LWrMot3, origin xyz=0 -0.049 -0.174 rpy=0 0 0, axis 0 0 1, limit lower=-2.55 upper=2.55 effort=27 velocity=6.283
- added joint RElbj: type revolute, parent RShy, child RElb, origin xyz=0.045 -0.05515 -0.074 rpy=0 0 0, axis 0 1 0, limit lower=-2.488 upper=0.292 effort=147 velocity=6.283
- added joint RForearmPlate: type revolute, parent RElb, child RForearm, origin xyz=-0.015 0.05515 -0.095 rpy=0 0 0, axis 0 0 1, limit lower=-2.55 upper=2.55 effort=55 velocity=6.283
- added joint RShLat: type revolute, parent RShp, child RShr, origin xyz=-0.09015 -0.062 0 rpy=0.1745327 0 0, axis 1 0 0, limit lower=-3.43 upper=-0.004 effort=120 velocity=6.283
- added joint RShSag: type revolute, parent DWYTorso, child RShp, origin xyz=0.0457475 -0.169137 0.155126 rpy=-0.174533 0 0.5235988, axis 0 1 0, limit lower=-3.359 upper=1.606 effort=147 velocity=6.283
- added joint RShYaw: type revolute, parent RShr, child RShy, origin xyz=0.09015 0 -0.21815 rpy=0 0 0, axis 0 0 1, limit lower=-2.55 upper=2.55 effort=147 velocity=6.283
- added joint RWrj1: type revolute, parent RForearm, child RWrMot2, origin xyz=0 -0.049 -0.156 rpy=0 0 0, axis 0 1 0, limit lower=-1.542 upper=1.508 effort=55 velocity=6.283
- added joint RWrj2: type revolute, parent RWrMot2, child RWrMot3, origin xyz=0 0.049 -0.174 rpy=0 0 0, axis 0 0 1, limit lower=-2.55 upper=2.55 effort=27 velocity=6.283
- added joint WaistFixed: type fixed, parent DWL, child DWLExt, origin xyz=-0.0540957 0.0 0.0635 rpy=0 0 0
- added joint WaistYaw: type revolute, parent DWLExt, child DWYTorso, origin xyz=0 0 0.16815 rpy=0 0 0, axis 0 0 1, limit lower=-1.74532925199 upper=1.74532925199 effort=120 velocity=6.283
- added joint imu_joint: type fixed, parent Waist, child imu_link, origin xyz=0 0 0 rpy=0 0 0
- joint LAnklePitch: limit lower=-0.872664625995 upper=0.698131700796 effort=179 velocity=4.9 -> lower=-0.872664625997 upper=0.698131700798 effort=179 velocity=4.9
- joint LAnkleRoll: limit lower=-0.261799387798 upper=0.261799387798 effort=230 velocity=3.2 -> lower=-0.261799387799 upper=0.261799387799 effort=230 velocity=3.2
- joint LHipLat: limit lower=-0.523598775597 upper=1.65806278939 effort=235 velocity=7.4 -> lower=-0.523598775598 upper=1.65806278939 effort=235 velocity=7.4
- joint LHipSag: limit lower=-1.91986217719 upper=1.55334303427 effort=235 velocity=7.4 -> lower=-1.91986217719 upper=1.55334303428 effort=235 velocity=7.4
- joint LHipYaw: limit lower=-0.558505360637 upper=1.57079632679 effort=153 velocity=4.6 -> lower=-0.558505360638 upper=1.5707963268 effort=153 velocity=4.6
- joint RAnklePitch: limit lower=-0.872664625995 upper=0.698131700796 effort=179 velocity=4.9 -> lower=-0.872664625997 upper=0.698131700798 effort=179 velocity=4.9
- joint RAnkleRoll: limit lower=-0.261799387798 upper=0.261799387798 effort=230 velocity=3.2 -> lower=-0.261799387799 upper=0.261799387799 effort=230 velocity=3.2
- joint RHipLat: limit lower=-1.65806278939 upper=0.523598775597 effort=235 velocity=7.4 -> lower=-1.65806278939 upper=0.523598775598 effort=235 velocity=7.4
- joint RHipSag: limit lower=-1.91986217719 upper=1.55334303427 effort=235 velocity=7.4 -> lower=-1.91986217719 upper=1.55334303428 effort=235 velocity=7.4
- joint RHipYaw: limit lower=-1.57079632679 upper=0.558505360637 effort=153 velocity=4.9 -> lower=-1.5707963268 upper=0.558505360638 effort=153 velocity=4.9
- joint WaistLat: limit lower=-0.523598775597 upper=0.523598775597 effort=150 velocity=7.4 -> lower=-0.523598775598 upper=0.523598775598 effort=150 velocity=7.4

Commit message: Added imu

File: iit-cogimon/model.urdf (robot description, URDF)
Before this commit: robot cogimon, 51 links, 50 joints
Links:
- link imu_link: mass 0 -> 0.01; geometry visual box size=0.01 0.01 0.01
