Commit message: fixed triangle foot model with corrected stl and naming for gazebo

File: kuka-lwr-4plus-triangle/model.urdf (robot description, URDF)
Before this commit: robot kuka-lwr-4plus-sponge, 11 links, 10 joints
Links:
- removed link lwr_ft_link
- link lwr_tool_link: mass 0.691 -> 0.355; geometry collision mesh filename=model://kuka-lwr-4plus-triangle/TriangleFoot.stl scale=0.01 0.01 0.01; visual mesh filename=model://kuka-lwr-4plus-triangle/TriangleFoot.stl scale=0.01 0.01 0.01
Joints:
- removed joint lwr_arm_ft_sensor_joint
- removed joint lwr_ft_sensor_tool_joint
- added joint lwr_arm_7_tool_joint: type fixed, parent lwr_arm_7_link, child lwr_tool_link, origin xyz=0 0 0.045 rpy=0 0 0, limit lower=0 upper=0 effort=0 velocity=0

Commit message: Fix tool orientation to avoid limit exceedance

File: kuka-lwr-4plus-triangle/model.urdf (robot description, URDF)
Before this commit: robot kuka-lwr-4plus-triangle, 10 links, 9 joints
Joints:
- joint lwr_arm_7_tool_joint: origin xyz=0 0 0.045 rpy=0 0 0 -> xyz=0 0 0.045 rpy=0 0 3.141592
