Commit message: new stuff

File: kuka-lwr-4plus-bh8-mod/model.urdf (robot description, URDF)
Before this commit: robot kuka-lwr-4plus-triangle, 10 links, 9 joints
Links:
- removed link lwr_tool_link
- link lwr_arm_base_link: geometry visual mesh filename=model://kuka-lwr-4plus/meshes/arm_base.dae scale=100 100 100
Joints:
- removed joint arm_world_joint
- removed joint lwr_arm_7_tool_joint
- added joint lwr_arm_world_joint: type fixed, parent world, child lwr_arm_base_link, origin xyz=0 0 0 rpy=0 0 0
