Commit message: added FT fix

File: BI-kuka-lwr-4plus-triangle-tilted-bh8-setup/model.urdf (robot description, URDF)
Before this commit: robot BI-kuka-lwr-4plus-triangle-tilted-bh8-setup, 45 links, 44 joints
Links:
- removed link left_bhand_palm_link
- removed link right_bhand_palm_link
- added link left/bhand_palm_link, mass 0.50573; collision box size=0.024 0.108 0.033; collision box size=0.076 0.046 0.012
- added link right/bhand_palm_link, mass 0.50573; collision box size=0.024 0.108 0.033; collision box size=0.076 0.046 0.012
Joints:
- joint left/finger_1/prox_joint: parent left_bhand_palm_link -> left/bhand_palm_link
- joint left/finger_2/prox_joint: parent left_bhand_palm_link -> left/bhand_palm_link
- joint left/finger_3/med_joint: parent left_bhand_palm_link -> left/bhand_palm_link
- joint left_bhand_grasp_joint: parent left_bhand_palm_link -> left/bhand_palm_link
- joint left_bhand_palm_surface_joint: parent left_bhand_palm_link -> left/bhand_palm_link
- joint left_lwr_arm_7_tool_joint: child left_bhand_palm_link -> left/bhand_palm_link; type revolute -> fixed
- joint right/finger_1/prox_joint: parent right_bhand_palm_link -> right/bhand_palm_link
- joint right/finger_2/prox_joint: parent right_bhand_palm_link -> right/bhand_palm_link
- joint right/finger_3/med_joint: parent right_bhand_palm_link -> right/bhand_palm_link
- joint right_bhand_grasp_joint: parent right_bhand_palm_link -> right/bhand_palm_link
- joint right_bhand_palm_surface_joint: parent right_bhand_palm_link -> right/bhand_palm_link
- joint right_lwr_arm_7_tool_joint: child right_bhand_palm_link -> right/bhand_palm_link; type revolute -> fixed

Commit message: new stuff

File: BI-kuka-lwr-4plus-triangle-tilted-bh8-setup/model.urdf (robot description, URDF)
Before this commit: robot BI-kuka-lwr-4plus-triangle-tilted-bh8-setup, 45 links, 44 joints
Links:
- added link left/compliance_link, mass 0.01; visual sphere radius=0.01
Joints:
- added joint left/compliance_joint: type fixed, parent left/bhand_palm_link, child left/compliance_link, origin xyz=0.0 0.0 0.18 rpy=0 0 0
