Commit message: advancements in iiwa and schunk models

File: kuka-iiwa-7-schunk-egp-40/model.urdf (robot description, URDF)
Before this commit: robot kuka-iiwa-7-schunk-egp-40, 12 links, 11 joints
Links:
- added link Tool_link
- link SchunkEGP40_Finger1_link: mass 1.0 -> 0.04
- link SchunkEGP40_Finger2_link: mass 1.0 -> 0.04
- link SchunkEGP40_link: mass 1.0 -> 0.6
Joints:
- added joint ee_tool_joint: type fixed, parent SchunkEGP40_link, child Tool_link, origin xyz=0 0 0.01215 rpy=0 0 0

File: schunk-egp-40/model.urdf (robot description, URDF)
Before this commit: robot schunk-egp-40, 3 links, 2 joints
Links:
- link SchunkEGP40_Finger1_link: mass 1.0 -> 0.04
- link SchunkEGP40_Finger2_link: mass 1.0 -> 0.04
- link SchunkEGP40_link: mass 1.0 -> 0.6

Commit message: updated inertia and mass

File: kuka-iiwa-7-schunk-egp-40/model.urdf (robot description, URDF)
Before this commit: robot kuka-iiwa-7-schunk-egp-40, 13 links, 12 joints
Links:
- removed link Tool_link
- link SchunkEGP40_Finger1_link: mass 0.04 -> 0.01
- link SchunkEGP40_Finger2_link: mass 0.04 -> 0.01
Joints:
- removed joint ee_tool_joint
